File: OriginalN64ExpansionPak.kicad_sch (KiCad schematic)
At the start: 14 parts, among them U1 MSM5718B70-60GS-K, U2 Expansion Pak Edge Connector

Commit message: Updating R13 to have a larger package size so it's easier to solder by hand
Parts:
- R13: value Yageo RC0603FR-07510RL -> Yageo RC0805FR-07510RL; footprint Resistor_SMD:R_0201_0603Metric -> Resistor_SMD:R_0805_2012Metric_Pad1.20x1.40mm_HandSolder; OCTOPART URL http://octopart.com/rc0603fr-07510rl-yageo-1403392 -> https://octopart.com/rc0805fr-07510rl-yageo-1169945?r=sp
Changed lines of the file:
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@@
       (effects (font (size 1.27 1.27)) (justify left bottom))
     )
-    (property "Value" "Yageo RC0603FR-07510RL" (id 1) (at 149.098 146.812 0)
-      (effects (font (size 1.27 1.27)) (justify left bottom) hide)
-    )
-    (property "Footprint" "Resistor_SMD:R_0201_0603Metric" (id 2) (at 152.4 149.86 0)
+    (property "Value" "Yageo RC0805FR-07510RL" (id 1) (at 149.098 146.812 0)
+      (effects (font (size 1.27 1.27)) (justify left bottom) hide)
+    )
+    (property "Footprint" "Resistor_SMD:R_0805_2012Metric_Pad1.20x1.40mm_HandSolder" (id 2) (at 152.4 149.86 0)
       (effects (font (size 1.27 1.27)) hide)
     )
@@
       (effects (font (size 1.27 1.27)) (justify left bottom) hide)
     )
-    (property "OCTOPART URL" "http://octopart.com/rc0603fr-07510rl-yageo-1403392" (id 5) (at 149.098 146.812 0)
+    (property "OCTOPART URL" "https://octopart.com/rc0805fr-07510rl-yageo-1169945?r=sp" (id 5) (at 149.098 146.812 0)
       (effects (font (size 1.27 1.27)) (justify left bottom) hide)
     )
@@
     )
     (path "/4e5b5311-d632-4381-8124-ee31df1f3492"
-      (reference "R13") (unit 1) (value "Yageo RC0603FR-07510RL") (footprint "Resistor_SMD:R_0201_0603Metric")
+      (reference "R13") (unit 1) (value "Yageo RC0805FR-07510RL") (footprint "Resistor_SMD:R_0805_2012Metric_Pad1.20x1.40mm_HandSolder")
     )
     (path "/543cc246-4a18-426d-b00c-ed2800181a8e"

Commit message: Updating resistor footprint
Parts:
- R13: CASE/PACKAGE 0603 -> 0805; LEAD-FREE STATUS Lead Free -> (none); MANUFACTURER PART NUMBER RC0603FR-07510RL -> (none); MOUNTING STYLE Surface Mount -> (none); OCTOPARTID c4ff0de08b991b38 -> (none); PACKAGING Tape & Reel (TR), Cut Tape (CT) -> (none); POWER RATING 100 mW -> (none); RESISTANCE TOLERANCE ±1% -> (none); ROHS Compliant -> (none); SELLER LANDING  URL https://octopart-clicks.com/click/track?country=US&ak=8157f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 -> (none); SIZE-HEIGHT 450 µm -> (none); SIZE-LENGTH 1.60 mm -> (none); SIZE-WIDTH 800 µm -> (none); VOLTAGE RATING (DC) 50.0 V -> (none)
Changed lines of the file:
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@@
       (effects (font (size 1.27 1.27)) (justify left bottom) hide)
     )
-    (property "MANUFACTURER PART NUMBER" "RC0603FR-07510RL" (id 6) (at 149.098 146.812 0)
+    (property "MANUFACTURER PART NUMBER" "" (id 6) (at 149.098 146.812 0)
       (effects (font (size 1.27 1.27)) (justify left bottom) hide)
     )
-    (property "SIZE-HEIGHT" "450 µm" (id 7) (at 149.098 146.812 0)
+    (property "SIZE-HEIGHT" "" (id 7) (at 149.098 146.812 0)
       (effects (font (size 1.27 1.27)) (justify left bottom) hide)
     )
-    (property "SELLER LANDING  URL" "https://octopart-clicks.com/click/track?country=US&ak=8157f166&sig=0faf81b&sid=1106&ppid=1403392&vpid=198667339&ct=offers" (id 8) (at 149.098 146.812 0)
+    (property "SELLER LANDING  URL" "" (id 8) (at 149.098 146.812 0)
       (effects (font (size 1.27 1.27)) (justify left bottom) hide)
     )
-    (property "LEAD-FREE STATUS" "Lead Free" (id 9) (at 149.098 146.812 0)
+    (property "LEAD-FREE STATUS" "" (id 9) (at 149.098 146.812 0)
       (effects (font (size 1.27 1.27)) (justify left bottom) hide)
     )
-    (property "OCTOPARTID" "c4ff0de08b991b38" (id 10) (at 149.098 146.812 0)
+    (property "OCTOPARTID" "" (id 10) (at 149.098 146.812 0)
       (effects (font (size 1.27 1.27)) (justify left bottom) hide)
     )
-    (property "MOUNTING STYLE" "Surface Mount" (id 11) (at 149.098 146.812 0)
+    (property "MOUNTING STYLE" "" (id 11) (at 149.098 146.812 0)
       (effects (font (size 1.27 1.27)) (justify left bottom) hide)
     )
-    (property "SIZE-WIDTH" "800 µm" (id 12) (at 149.098 146.812 0)
+    (property "SIZE-WIDTH" "" (id 12) (at 149.098 146.812 0)
       (effects (font (size 1.27 1.27)) (justify left bottom) hide)
     )
-    (property "VOLTAGE RATING (DC)" "50.0 V" (id 13) (at 149.098 146.812 0)
+    (property "VOLTAGE RATING (DC)" "" (id 13) (at 149.098 146.812 0)
       (effects (font (size 1.27 1.27)) (justify left bottom) hide)
     )
-    (property "SIZE-LENGTH" "1.60 mm" (id 14) (at 149.098 146.812 0)
+    (property "SIZE-LENGTH" "" (id 14) (at 149.098 146.812 0)
       (effects (font (size 1.27 1.27)) (justify left bottom) hide)
     )
@@
       (effects (font (size 1.27 1.27)) (justify left bottom))
     )
-    (property "CASE/PACKAGE" "0603" (id 16) (at 149.098 146.812 0)
+    (property "CASE/PACKAGE" "0805" (id 16) (at 149.098 146.812 0)
       (effects (font (size 1.27 1.27)) (justify left bottom) hide)
     )
-    (property "ROHS" "Compliant" (id 17) (at 149.098 146.812 0)
+    (property "ROHS" "" (id 17) (at 149.098 146.812 0)
       (effects (font (size 1.27 1.27)) (justify left bottom) hide)
     )
-    (property "PACKAGING" "Tape & Reel (TR), Cut Tape (CT)" (id 18) (at 149.098 146.812 0)
+    (property "PACKAGING" "" (id 18) (at 149.098 146.812 0)
       (effects (font (size 1.27 1.27)) (justify left bottom) hide)
     )
-    (property "RESISTANCE TOLERANCE" "±1%" (id 19) (at 149.098 146.812 0)
+    (property "RESISTANCE TOLERANCE" "" (id 19) (at 149.098 146.812 0)
       (effects (font (size 1.27 1.27)) (justify left bottom) hide)
     )
-    (property "POWER RATING" "100 mW" (id 20) (at 149.098 146.812 0)
+    (property "POWER RATING" "" (id 20) (at 149.098 146.812 0)
       (effects (font (size 1.27 1.27)) (justify left bottom) hide)
     )
