File: OriginalN64ExpansionPak.kicad_pcb (KiCad board)
At the start: 2 copper layers, 41.9 x 21 mm, 14 parts, among them U1 MSM5718B70-60GS-K, U2 Expansion Pak Edge Connector

Commit message: Updating solder pads to be 'Hand_Solder' variants to make soldering less painful. Also updated how the copper pours interact with the edge connector
Parts:
- C1, C2, C3, C4, C5, C6, C7, C8: footprint Capacitor_SMD:C_0805_2012Metric -> Capacitor_SMD:C_0805_2012Metric_Pad1.18x1.45mm_HandSolder
